File: AS3340_VCO/file5D38223D.sch (KiCad schematic (older format))
At the start: 29 parts, among them U2 TL071

Commit message: AS3340_VCO rev 2 AS3310_ADSR rev 1 AS3320_VCF rev 1 AS3360_VCA rev 1 ER_Bus_Board rev 1
Parts:
- removed R13: 1M, Resistor_SMD:R_0805_2012Metric, symbol Device:R_US
- removed RV3: 20K, Potentiometer_THT:Potentiometer_Bourns_3296W_Vertical, symbol Device:R_POT_TRIM_US
- added R40: 22K, Resistor_SMD:R_0805_2012Metric, symbol Device:R_US
- added R41: 100K, Resistor_SMD:R_0805_2012Metric, symbol Device:R_US
- added R42: 1M, Resistor_SMD:R_0805_2012Metric, symbol Device:R_US
- added RV13: 100K, Potentiometer_THT:Potentiometer_Bourns_3296W_Vertical, symbol Device:R_POT_TRIM_US
- added RV14: 10K, Potentiometer_THT:Potentiometer_Bourns_3296W_Vertical, symbol Device:R_POT_TRIM_US
- R14: value 360K -> 100K
- R21: value 1.5M -> 1.2M
- U2: footprint Package_SO:SOIC-8_3.9x4.9mm_P1.27mm -> Package_DIP:DIP-8_W7.62mm
Connections:
- net +12V: now also RV13.1, RV14.1; no longer R14.1, R21.2
- net CV: now also R41.1, R42.1; no longer RV4.2, RV5.2
- net GNDREF: now also R40.1
- new net: R41.2, RV4.2
- new net: R42.2, RV5.2
- new net: R14.1, RV13.2, RV13.3
- new net: R21.2, RV14.2
- new net: R40.2, RV14.3
Other:
- note removed: "High Freq. Tracking Trim"
- moved on the sheet: R16, R17, R18, R19, RV4, RV5
