File: AS3340_VCO/file5D2AE37E.sch (KiCad schematic (older format))
At the start: 26 parts, among them U4 TL071, U5 LM13700, U6 TL072

Commit message: AS3340_VCO rev 2 AS3310_ADSR rev 1 AS3320_VCF rev 1 AS3360_VCA rev 1 ER_Bus_Board rev 1
Parts:
- U4, U6: footprint Package_SO:SOIC-8_3.9x4.9mm_P1.27mm -> Package_DIP:DIP-8_W7.62mm
- U5: footprint Package_SO:SOIC-16_3.9x9.9mm_P1.27mm -> Package_DIP:DIP-16_W7.62mm
Changed lines of the file:
@@
 F 0 "U5" H 4700 1767 50  0000 C CNN
 F 1 "LM13700" H 4700 1676 50  0000 C CNN
-F 2 "Package_SO:SOIC-16_3.9x9.9mm_P1.27mm" H 4400 1425 50  0001 C CNN
+F 2 "Package_DIP:DIP-16_W7.62mm" H 4400 1425 50  0001 C CNN
 F 3 "http://www.ti.com/lit/ds/symlink/lm13700.pdf" H 4400 1425 50  0001 C CNN
 	3    4700 1400
@@
 F 0 "U5" H 5750 1748 50  0000 C CNN
 F 1 "LM13700" H 5750 1657 50  0000 C CNN
-F 2 "Package_SO:SOIC-16_3.9x9.9mm_P1.27mm" H 5550 1425 50  0001 C CNN
+F 2 "Package_DIP:DIP-16_W7.62mm" H 5550 1425 50  0001 C CNN
 F 3 "http://www.ti.com/lit/ds/symlink/lm13700.pdf" H 5550 1425 50  0001 C CNN
 	4    5850 1400
@@
 F 0 "U5" H 9558 4096 50  0000 L CNN
 F 1 "LM13700" H 9558 4005 50  0000 L CNN
-F 2 "Package_SO:SOIC-16_3.9x9.9mm_P1.27mm" H 9300 4075 50  0001 C CNN
+F 2 "Package_DIP:DIP-16_W7.62mm" H 9300 4075 50  0001 C CNN
 F 3 "http://www.ti.com/lit/ds/symlink/lm13700.pdf" H 9300 4075 50  0001 C CNN
 	5    9600 4050
@@
 F 0 "U6" H 2650 7017 50  0000 C CNN
 F 1 "TL072" H 2650 6926 50  0000 C CNN
-F 2 "Package_SO:SOIC-8_3.9x4.9mm_P1.27mm" H 2650 6650 50  0001 C CNN
+F 2 "Package_DIP:DIP-8_W7.62mm" H 2650 6650 50  0001 C CNN
 F 3 "http://www.ti.com/lit/ds/symlink/tl071.pdf" H 2650 6650 50  0001 C CNN
 	1    2650 6650
@@
 F 0 "U6" H 5650 7017 50  0000 C CNN
 F 1 "TL072" H 5650 6926 50  0000 C CNN
-F 2 "Package_SO:SOIC-8_3.9x4.9mm_P1.27mm" H 5650 6650 50  0001 C CNN
+F 2 "Package_DIP:DIP-8_W7.62mm" H 5650 6650 50  0001 C CNN
 F 3 "http://www.ti.com/lit/ds/symlink/tl071.pdf" H 5650 6650 50  0001 C CNN
 	2    5650 6650
@@
 F 0 "U6" H 9058 4096 50  0000 L CNN
 F 1 "TL072" H 9058 4005 50  0000 L CNN
-F 2 "Package_SO:SOIC-8_3.9x4.9mm_P1.27mm" H 9100 4050 50  0001 C CNN
+F 2 "Package_DIP:DIP-8_W7.62mm" H 9100 4050 50  0001 C CNN
 F 3 "http://www.ti.com/lit/ds/symlink/tl071.pdf" H 9100 4050 50  0001 C CNN
 	3    9100 4050
@@
 F 0 "U4" H 3150 3750 50  0000 L CNN
 F 1 "TL071" H 3150 3650 50  0000 L CNN
-F 2 "Package_SO:SOIC-8_3.9x4.9mm_P1.27mm" H 3050 3550 50  0001 C CNN
+F 2 "Package_DIP:DIP-8_W7.62mm" H 3050 3550 50  0001 C CNN
 F 3 "http://www.ti.com/lit/ds/symlink/tl071.pdf" H 3150 3650 50  0001 C CNN
 	1    3000 3500
@@
 F 0 "U5" H 9850 2867 50  0000 C CNN
 F 1 "LM13700" H 9850 2776 50  0000 C CNN
-F 2 "Package_SO:SOIC-16_3.9x9.9mm_P1.27mm" H 9550 2525 50  0001 C CNN
+F 2 "Package_DIP:DIP-16_W7.62mm" H 9550 2525 50  0001 C CNN
 F 3 "http://www.ti.com/lit/ds/symlink/lm13700.pdf" H 9550 2525 50  0001 C CNN
 	1    9850 2500
@@
 F 0 "U5" H 9950 2048 50  0000 C CNN
 F 1 "LM13700" H 9950 1957 50  0000 C CNN
-F 2 "Package_SO:SOIC-16_3.9x9.9mm_P1.27mm" H 9750 1725 50  0001 C CNN
+F 2 "Package_DIP:DIP-16_W7.62mm" H 9750 1725 50  0001 C CNN
 F 3 "http://www.ti.com/lit/ds/symlink/lm13700.pdf" H 9750 1725 50  0001 C CNN
 	2    10050 1700

Commit message: Re-do VCO board to support new front panel board
Parts:
- removed U4: TL071, Package_DIP:DIP-8_W7.62mm, symbol Amplifier_Operational:TL071
- added R12, R14: 10K, Resistor_SMD:R_0805_2012Metric, symbol Device:R_US
- added U7: TL072, Package_DIP:DIP-8_W7.62mm, symbol Amplifier_Operational:TL072
Connections:
- net +12V: now also U7.8 (V+)
- net -12V: now also U7.4 (V-)
- net GNDREF: now also U6.5 (+)
- net PULSE: now also U7.7; no longer U6.7
- net SAW: now also R12.1
- net TRI: now also U7.1
- net at RV11.2: now also U7.5 (+); no longer U6.5 (+)
- net at R38.2, R39.1: now also U7.6 (-); no longer U6.6 (-)
- net at R24.2, R25.1: now also U7.2 (-)
- net at RV6.2: now also U7.3 (+)
- net RAW_SAW renamed RAW_RAMP
- new net: R12.2, R14.1, U6.6 (-)
- new net RAMP: R14.2, U6.7
- no-connect marks 2 -> 0
Other:
- moved on the sheet: R37, R38, R39, RV11, U6B
