File: VCA/Front_Panel/VCA_Front_Panel.sch (KiCad schematic (older format))
At the start: 1 part

Commit message: Bunch of bug fixes and tweaks
Parts:
- removed TP1: TestPoint, TestPoint:TestPoint_Pad_1.0x1.0mm, symbol Connector:TestPoint
- added H1: Level_A, Eurorack:pot_fp_hole, symbol Mechanical:MountingHole_Pad
- added H10: In_B, Eurorack:jack_fp_hole, symbol Mechanical:MountingHole_Pad
- added H11: Out_A, Eurorack:jack_fp_hole, symbol Mechanical:MountingHole_Pad
- added H12: Out_B, Eurorack:jack_fp_hole, symbol Mechanical:MountingHole_Pad
- added H13: Top_MH, Eurorack:eurorack_mounting_hole, symbol Mechanical:MountingHole_Pad
- added H14: Bottom_MH, Eurorack:eurorack_mounting_hole, symbol Mechanical:MountingHole_Pad
- added H2: Level_B, Eurorack:pot_fp_hole, symbol Mechanical:MountingHole_Pad
- added H3: Lin_Log_A, Eurorack:jack_fp_hole, symbol Mechanical:MountingHole_Pad
- added H4: Lin_Log_B, Eurorack:jack_fp_hole, symbol Mechanical:MountingHole_Pad
- added H5: CV1_A, Eurorack:jack_fp_hole, symbol Mechanical:MountingHole_Pad
- added H6: CV1_B, Eurorack:jack_fp_hole, symbol Mechanical:MountingHole_Pad
- added H7: CV2_A, Eurorack:jack_fp_hole, symbol Mechanical:MountingHole_Pad
- added H8: CV2_B, Eurorack:jack_fp_hole, symbol Mechanical:MountingHole_Pad
- added H9: In_A, Eurorack:jack_fp_hole, symbol Mechanical:MountingHole_Pad
Connections:
- wire segments 2 -> 0
