File: VCO/Front_Panel/VCO_Front_Panel.sch (KiCad schematic (older format))
At the start: 1 part

Commit message: Bunch of bug fixes and tweaks
Parts:
- removed TP1: TestPoint, TestPoint:TestPoint_Pad_1.0x1.0mm, symbol Connector:TestPoint
- added H1: Top_MH1, Eurorack:eurorack_mounting_hole, symbol Mechanical:MountingHole_Pad
- added H10: Ramp, Eurorack:jack_fp_hole, symbol Mechanical:MountingHole_Pad
- added H11: Saw, Eurorack:jack_fp_hole, symbol Mechanical:MountingHole_Pad
- added H12: PWM_Mod, Eurorack:jack_fp_hole, symbol Mechanical:MountingHole_Pad
- added H13: CV1, Eurorack:jack_fp_hole, symbol Mechanical:MountingHole_Pad
- added H14: Tri, Eurorack:jack_fp_hole, symbol Mechanical:MountingHole_Pad
- added H15: CV2, Eurorack:jack_fp_hole, symbol Mechanical:MountingHole_Pad
- added H16: Sine, Eurorack:jack_fp_hole, symbol Mechanical:MountingHole_Pad
- added H17: CV3, Eurorack:jack_fp_hole, symbol Mechanical:MountingHole_Pad
- added H18: Top_MH2, Eurorack:eurorack_mounting_hole, symbol Mechanical:MountingHole_Pad
- added H19: Bottom_MH2, Eurorack:eurorack_mounting_hole, symbol Mechanical:MountingHole_Pad
- added H2: Bottom_MH1, Eurorack:eurorack_mounting_hole, symbol Mechanical:MountingHole_Pad
- added H3: Coarse, Eurorack:pot_fp_hole, symbol Mechanical:MountingHole_Pad
- added H4: PWM_Amt, Eurorack:pot_fp_hole, symbol Mechanical:MountingHole_Pad
- added H5: Sync, Eurorack:jack_fp_hole, symbol Mechanical:MountingHole_Pad
- added H6: Pulse, Eurorack:jack_fp_hole, symbol Mechanical:MountingHole_Pad
- added H7: Fine, Eurorack:pot_fp_hole, symbol Mechanical:MountingHole_Pad
- added H8: PWM_Width, Eurorack:pot_fp_hole, symbol Mechanical:MountingHole_Pad
- added H9: Lin, Eurorack:jack_fp_hole, symbol Mechanical:MountingHole_Pad
Connections:
- wire segments 2 -> 0
