File: VCF/IO/VCF_IO.sch (KiCad schematic (older format))
At the start: 14 parts, among them J1 Res Mod, J2 Cutoff Mod, J3 In1, J4 In2, J5 In3, J6 Out, J7 IO

Commit message: Fix inverted resonance control input
Connections:
- net +12V: now also RV6.1
- net -12V: no longer RV6.1
Changed lines of the file:
@@
 Wire Wire Line
 	4900 2200 5400 2200
-$Comp
-L power:-12V #PWR0113
-U 1 1 5D91479A
-P 4900 2900
-F 0 "#PWR0113" H 4900 3000 50  0001 C CNN
-F 1 "-12V" H 4915 3073 50  0000 C CNN
-F 2 "" H 4900 2900 50  0001 C CNN
-F 3 "" H 4900 2900 50  0001 C CNN
-	1    4900 2900
-	-1   0    0    1
-$EndComp
 Wire Wire Line
 	4900 3250 5400 3250
@@
 Text Label 7700 2900 0    50   ~ 0
 Out
+$Comp
+L power:+12V #PWR?
+U 1 1 5D8D5D9B
+P 4750 2950
+F 0 "#PWR?" H 4750 2800 50  0001 C CNN
+F 1 "+12V" H 4765 3123 50  0000 C CNN
+F 2 "" H 4750 2950 50  0001 C CNN
+F 3 "" H 4750 2950 50  0001 C CNN
+	1    4750 2950
+	1    0    0    -1
+$EndComp
 Wire Wire Line
-	4750 2800 4900 2800
-Wire Wire Line
-	4900 2800 4900 2900
-Wire Wire Line
-	4750 2800 4750 3100
+	4750 2950 4750 3100
 $EndSCHEMATC

Commit message: Bunch of bug fixes and tweaks
Parts:
- added H1: Top_MH1, Eurorack:eurorack_mounting_hole, symbol Mechanical:MountingHole_Pad
- added H2: Bottom_MH1, Eurorack:eurorack_mounting_hole, symbol Mechanical:MountingHole_Pad
- added H3: Top_MH2, Eurorack:eurorack_mounting_hole, symbol Mechanical:MountingHole_Pad
- added H4: Bottom_MH2, Eurorack:eurorack_mounting_hole, symbol Mechanical:MountingHole_Pad
Connections:
- net GNDREF: now also H1.1, H2.1, H3.1, H4.1
Changed lines of the file:
@@
 Out
 $Comp
-L power:+12V #PWR?
+L power:+12V #PWR01
 U 1 1 5D8D5D9B
 P 4750 2950
-F 0 "#PWR?" H 4750 2800 50  0001 C CNN
+F 0 "#PWR01" H 4750 2800 50  0001 C CNN
 F 1 "+12V" H 4765 3123 50  0000 C CNN
 F 2 "" H 4750 2950 50  0001 C CNN
@@
 Wire Wire Line
 	4750 2950 4750 3100
+$Comp
+L Mechanical:MountingHole_Pad H1
+U 1 1 5D92F84E
+P 5900 850
+F 0 "H1" H 6000 899 50  0000 L CNN
+F 1 "Top_MH1" H 6000 808 50  0000 L CNN
+F 2 "Eurorack:eurorack_mounting_hole" H 5900 850 50  0001 C CNN
+F 3 "~" H 5900 850 50  0001 C CNN
+	1    5900 850
+	1    0    0    -1
+$EndComp
+$Comp
+L power:GNDREF #PWR02
+U 1 1 5D92FCB3
+P 5900 950
+F 0 "#PWR02" H 5900 700 50  0001 C CNN
+F 1 "GNDREF" H 5905 777 50  0001 C CNN
+F 2 "" H 5900 950 50  0001 C CNN
+F 3 "" H 5900 950 50  0001 C CNN
+	1    5900 950
+	1    0    0    -1
+$EndComp
+$Comp
+L Mechanical:MountingHole_Pad H3
+U 1 1 5D930C42
+P 6750 850
+F 0 "H3" H 6850 899 50  0000 L CNN
+F 1 "Top_MH2" H 6850 808 50  0000 L CNN
+F 2 "Eurorack:eurorack_mounting_hole" H 6750 850 50  0001 C CNN
+F 3 "~" H 6750 850 50  0001 C CNN
+	1    6750 850
+	1    0    0    -1
+$EndComp
+$Comp
+L power:GNDREF #PWR04
+U 1 1 5D930C48
+P 6750 950
+F 0 "#PWR04" H 6750 700 50  0001 C CNN
+F 1 "GNDREF" H 6755 777 50  0001 C CNN
+F 2 "" H 6750 950 50  0001 C CNN
+F 3 "" H 6750 950 50  0001 C CNN
+	1    6750 950
+	1    0    0    -1
+$EndComp
+$Comp
+L Mechanical:MountingHole_Pad H2
+U 1 1 5D931DD2
+P 5900 1250
+F 0 "H2" H 6000 1299 50  0000 L CNN
+F 1 "Bottom_MH1" H 6000 1208 50  0000 L CNN
+F 2 "Eurorack:eurorack_mounting_hole" H 5900 1250 50  0001 C CNN
+F 3 "~" H 5900 1250 50  0001 C CNN
+	1    5900 1250
+	1    0    0    -1
+$EndComp
+$Comp
+L power:GNDREF #PWR03
+U 1 1 5D931DD8
+P 5900 1350
+F 0 "#PWR03" H 5900 1100 50  0001 C CNN
+F 1 "GNDREF" H 5905 1177 50  0001 C CNN
+F 2 "" H 5900 1350 50  0001 C CNN
+F 3 "" H 5900 1350 50  0001 C CNN
+	1    5900 1350
+	1    0    0    -1
+$EndComp
+$Comp
+L Mechanical:MountingHole_Pad H4
+U 1 1 5D932EC2
+P 6750 1250
+F 0 "H4" H 6850 1299 50  0000 L CNN
+F 1 "Bottom_MH2" H 6850 1208 50  0000 L CNN
+F 2 "Eurorack:eurorack_mounting_hole" H 6750 1250 50  0001 C CNN
+F 3 "~" H 6750 1250 50  0001 C CNN
+	1    6750 1250
+	1    0    0    -1
+$EndComp
+$Comp
+L power:GNDREF #PWR05
+U 1 1 5D932EC8
+P 6750 1350
+F 0 "#PWR05" H 6750 1100 50  0001 C CNN
+F 1 "GNDREF" H 6755 1177 50  0001 C CNN
+F 2 "" H 6750 1350 50  0001 C CNN
+F 3 "" H 6750 1350 50  0001 C CNN
+	1    6750 1350
+	1    0    0    -1
+$EndComp
 $EndSCHEMATC

Commit message: Make VCF front panel bigger. Re-align IO and FP boards.
Parts:
- J1: value Res Mod -> Out
- J6: value Out -> Res Mod
Changed lines of the file:
@@
 P 5900 4050
 F 0 "J1" H 5932 4375 50  0000 C CNN
-F 1 "Res Mod" H 5932 4284 50  0000 C CNN
+F 1 "Out" H 5932 4284 50  0000 C CNN
 F 2 "Eurorack:Jack_3.5mm_QingPu_WQP-PJ398SM_Vertical_CircularHoles" H 5900 4050 50  0001 C CNN
 F 3 "~" H 5900 4050 50  0001 C CNN
@@
 P 2600 2950
 F 0 "J6" H 2632 3275 50  0000 C CNN
-F 1 "Out" H 2632 3184 50  0000 C CNN
+F 1 "Res Mod" H 2632 3184 50  0000 C CNN
 F 2 "Eurorack:Jack_3.5mm_QingPu_WQP-PJ398SM_Vertical_CircularHoles" H 2600 2950 50  0001 C CNN
 F 3 "~" H 2600 2950 50  0001 C CNN

Commit message: Fix backwards knobs
Connections:
- net +12V: now also RV1.3, RV6.3; no longer RV1.1, RV6.1
- net GNDREF: now also RV1.1, RV2.1, RV3.1, RV4.1, RV5.1, RV6.1, RV7.1; no longer RV1.3, RV2.3, RV3.3, RV4.3, RV5.3, RV6.3, RV7.3
- net at J2.T: now also RV4.3; no longer RV4.1
- net at J3.T: now also RV2.3; no longer RV2.1
- net at J4.T: now also RV3.3; no longer RV3.1
- net at J5.T: now also RV5.3; no longer RV5.1
- net at J6.T: now also RV7.3; no longer RV7.1
Changed lines of the file:
@@
 F 3 "~" H 3100 2200 50  0001 C CNN
 	1    3100 2200
-	1    0    0    -1
+	1    0    0    1
 $EndComp
 $Comp
@@
 F 3 "~" H 4750 2200 50  0001 C CNN
 	1    4750 2200
-	1    0    0    -1
+	1    0    0    1
 $EndComp
 $Comp
@@
 F 3 "~" H 3100 4100 50  0001 C CNN
 	1    3100 4100
-	1    0    0    -1
+	1    0    0    1
 $EndComp
 $Comp
@@
 F 3 "~" H 3100 5000 50  0001 C CNN
 	1    3100 5000
-	1    0    0    -1
+	1    0    0    1
 $EndComp
 $Comp
@@
 F 3 "~" H 3100 5950 50  0001 C CNN
 	1    3100 5950
-	1    0    0    -1
+	1    0    0    1
 $EndComp
 $Comp
@@
 F 3 "~" H 4750 3250 50  0001 C CNN
 	1    4750 3250
-	1    0    0    -1
+	1    0    0    1
 $EndComp
 $Comp
@@
 F 3 "~" H 3100 3250 50  0001 C CNN
 	1    3100 3250
-	1    0    0    -1
-$EndComp
-Wire Wire Line
+	1    0    0    1
+$EndComp
+Wire Wire Line
